File: Sofle_Pico/PCB/Sofle_Pico.kicad_sch (KiCad schematic)
At the start: 116 parts, among them J1 Conn_01x05, J2 MJ-4PP-9, J3 Conn_01x04, J4 Conn_01x04, J5 Conn_02x05_Odd_Even, J7 Conn_01x04, Q1 Si2301CDS, SW1 SW_PUSH, SW10 SW_PUSH, SW11 SW_PUSH, SW12 SW_PUSH, SW13 SW_PUSH, SW14 SW_PUSH, SW15 SW_PUSH, SW16 SW_PUSH, SW17 SW_PUSH, SW18 SW_PUSH, SW19 SW_PUSH, SW2 SW_PUSH, SW20 SW_PUSH, SW21 SW_PUSH, SW22 SW_PUSH, SW23 SW_PUSH, SW24 SW_PUSH, SW25 Rotary_Encoder_Switch-Device, SW26 SW_PUSH, SW27 SW_PUSH, SW28 SW_PUSH, SW29 SW_PUSH, SW3 SW_PUSH, SW30 SW_PUSH, SW4 SW_PUSH, SW5 SW_PUSH, SW6 SW_PUSH, SW7 SW_PUSH, SW8 SW_PUSH, SW9 SW_PUSH, U2 Pico

Commit message: Upgrade to kicad 9.0 project and fix name in schematic to remove choc.
Parts:
- D31: value MBR120VLSF -> MBR120VLSF
Other:
- title: Sofle Pico Choc -> Sofle Pico
Changed lines of the file:
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@@
 (kicad_sch
-	(version 20231120)
+	(version 20250114)
 	(generator "eeschema")
-	(generator_version "8.0")
+	(generator_version "9.0")
 	(paper "A")
 	(title_block
-		(title "Sofle Pico Choc")
-		(date "2024-07-04")
+		(title "Sofle Pico")
+		(date "2025-10-23")
 		(rev "v3.5.6")
 		(comment 1 "https://github.com/josefadamcik/SofleKeyboard")
@@
 		(comment 4 "Designed by Ryan Neff, Choc'd by P. Werle")
 	)
+	(rectangle
+		(start 15.24 90.17)
+		(end 39.37 106.68)
+		(stroke
+			(width 0)
+			(type default)
+		)
+		(fill
+			(type none)
+		)
+	)
+	(rectangle
+		(start 41.91 90.17)
+		(end 66.04 106.68)
+		(stroke
+			(width 0)
+			(type default)
+		)
+		(fill
+			(type none)
+		)
+	)
+	(rectangle
+		(start 15.24 119.38)
+		(end 62.23 143.51)
+		(stroke
+			(width 0)
+			(type default)
+		)
+		(fill
+			(type none)
+		)
+	)
+	(rectangle
+		(start 67.31 119.38)
+		(end 129.54 143.51)
+		(stroke
+			(width 0)
+			(type default)
+		)
+		(fill
+			(type none)
+		)
+	)
+	(rectangle
+		(start 74.93 90.17)
+		(end 99.06 106.68)
+		(stroke
+			(width 0)
+			(type default)
+		)
+		(fill
+			(type none)
+		)
+	)
+	(rectangle
+		(start 15.24 147.32)
+		(end 93.98 171.45)
+		(stroke
+			(width 0)
+			(type default)
+		)
+		(fill
+			(type none)
+		)
+	)
+	(text "Cirque trackpad RH (Optional)\n"
+		(exclude_from_sim no)
+		(at 41.91 88.9 0)
+		(effects
+			(font
+				(size 1.27 1.27)
+			)
+			(justify left bottom)
+		)
+	)
+	(text "I2C Pull-Ups "
+		(exclude_from_sim no)
+		(at 106.68 88.9 0)
+		(effects
+			(font
+				(size 1.27 1.27)
+			)
+			(justify left bottom)
+		)
+	)
+	(text "TRRS jack. full duplex with TX RX crossover in config \nis the default. (SERIAL_USART_FULL_DUPLEX)\nIf you really need an extra pin, \nyou can reconfigure for Serial with TX only."
+		(exclude_from_sim no)
+		(at 68.58 118.11 0)
+		(effects
+			(font
+				(size 1.27 1.27)
+			)
+			(justify left bottom)
+		)
+	)
+	(text "Rotary encoder, EC11 or EC12 (Optional)\n"
+		(exclude_from_sim no)
+		(at 15.24 118.11 0)
+		(effects
+			(font
+				(size 1.27 1.27)
+			)
+			(justify left bottom)
+		)
+	)
+	(text "D31 is not required for RPI Pico SCH compliant \nboards that have an onboard Schottky Diode.\nRefer to Sofle-Pico build guide \nand your RPI Module Datasheet/SCH. \n\nVSYS is variable depending on diode used! \nUser MUST know/verify whether or not their \nMCU Module is pin compliant with RPI Pico. \nRead RPI Pico datasheet Chapter 4.5-4.6\n\nVSYS≈4.9-5.0V w/ USB Power\nVSYS≈4.7-4.9V w/ TRRS Power"
+		(exclude_from_sim no)
+		(at 84.582 43.688 0)
+		(effects
+			(font
+				(size 1.27 1.27)
+			)
+			(justify left bottom)
+		)
+	)
+	(text "OPTIONAL:\nSplit Master Assignment\nInstall Resistor value ~2.2-10k\nR4 3.3V = LEFT\nR3 GND = RIGHT"
+		(exclude_from_sim no)
+		(at 105.156 76.708 0)
+		(effects
+			(font
+				(size 1.27 1.27)
+			)
+			(justify left bottom)
+		)
+	)
+	(text "OLEDs(Optional)\n"
+		(exclude_from_sim no)
+		(at 15.24 88.9 0)
+		(effects
+			(font
+				(size 1.27 1.27)
+			)
+			(justify left bottom)
+		)
+	)
+	(text "Patch Bay"
+		(exclude_from_sim no)
+		(at 15.24 147.32 0)
+		(effects
+			(font
+				(size 1.27 1.27)
+			)
+			(justify left bottom)
+		)
+	)
+	(text "Cirque trackpad LH (Optional)\n"
+		(exclude_from_sim no)
+		(at 74.93 88.9 0)
+		(effects
+			(font
+				(size 1.27 1.27)
+			)
+			(justify left bottom)
+		)
+	)
+	(text "OPTIONAL decoupling 0805\n"
+		(exclude_from_sim no)
+		(at 88.265 50.165 0)
+		(effects
+			(font
+				(size 1.27 1.27)
+			)
+			(justify left bottom)
+		)
+	)
+	(text "3.5.5 SCH Change Notes:\nI2C Pin Heaqders power pin now 3V3 \nAdded GND pin to J5.5  \nAll spare GPIO to patch bay"
+		(exclude_from_sim no)
+		(at 15.24 180.34 0)
+		(effects
+			(font
+				(size 1.27 1.27)
+			)
+			(justify left bottom)
+			(href "#1")
+		)
+	)
 	(junction
 		(at 179.07 163.83)
@@
 		)
 	)
-	(rectangle
-		(start 15.24 90.17)
-		(end 39.37 106.68)
-		(stroke
-			(width 0)
-			(type default)
-		)
-		(fill
-			(type none)
-		)
-	)
-	(rectangle
-		(start 41.91 90.17)
-		(end 66.04 106.68)
-		(stroke
-			(width 0)
-			(type default)
-		)
-		(fill
-			(type none)
-		)
-	)
-	(rectangle
-		(start 15.24 119.38)
-		(end 62.23 143.51)
-		(stroke
-			(width 0)
-			(type default)
-		)
-		(fill
-			(type none)
-		)
-	)
-	(rectangle
-		(start 67.31 119.38)
-		(end 129.54 143.51)
-		(stroke
-			(width 0)
-			(type default)
-		)
-		(fill
-			(type none)
-		)
-	)
-	(rectangle
-		(start 74.93 90.17)
-		(end 99.06 106.68)
-		(stroke
-			(width 0)
-			(type default)
-		)
-		(fill
-			(type none)
-		)
-	)
-	(rectangle
-		(start 15.24 147.32)
-		(end 93.98 171.45)
-		(stroke
-			(width 0)
-			(type default)
-		)
-		(fill
-			(type none)
-		)
-	)
-	(text "Cirque trackpad RH (Optional)\n"
-		(exclude_from_sim no)
-		(at 41.91 88.9 0)
-		(effects
-			(font
-				(size 1.27 1.27)
-			)
-			(justify left bottom)
-		)
-	)
-	(text "I2C Pull-Ups "
-		(exclude_from_sim no)
-		(at 106.68 88.9 0)
-		(effects
-			(font
-				(size 1.27 1.27)
-			)
-			(justify left bottom)
-		)
-	)
-	(text "TRRS jack. full duplex with TX RX crossover in config \nis the default. (SERIAL_USART_FULL_DUPLEX)\nIf you really need an extra pin, \nyou can reconfigure for Serial with TX only."
-		(exclude_from_sim no)
-		(at 68.58 118.11 0)
-		(effects
-			(font
-				(size 1.27 1.27)
-			)
-			(justify left bottom)
-		)
-	)
-	(text "Rotary encoder, EC11 or EC12 (Optional)\n"
-		(exclude_from_sim no)
-		(at 15.24 118.11 0)
-		(effects
-			(font
-				(size 1.27 1.27)
-			)
-			(justify left bottom)
-		)
-	)
-	(text "D31 is not required for RPI Pico SCH compliant \nboards that have an onboard Schottky Diode.\nRefer to Sofle-Pico build guide \nand your RPI Module Datasheet/SCH. \n\nVSYS is variable depending on diode used! \nUser MUST know/verify whether or not their \nMCU Module is pin compliant with RPI Pico. \nRead RPI Pico datasheet Chapter 4.5-4.6\n\nVSYS≈4.9-5.0V w/ USB Power\nVSYS≈4.7-4.9V w/ TRRS Power"
-		(exclude_from_sim no)
-		(at 84.582 43.688 0)
-		(effects
-			(font
-				(size 1.27 1.27)
-			)
-			(justify left bottom)
-		)
-	)
-	(text "OPTIONAL:\nSplit Master Assignment\nInstall Resistor value ~2.2-10k\nR4 3.3V = LEFT\nR3 GND = RIGHT"
-		(exclude_from_sim no)
-		(at 105.156 76.708 0)
-		(effects
-			(font
-				(size 1.27 1.27)
-			)
-			(justify left bottom)
-		)
-	)
-	(text "OLEDs(Optional)\n"
-		(exclude_from_sim no)
-		(at 15.24 88.9 0)
-		(effects
-			(font
-				(size 1.27 1.27)
-			)
-			(justify left bottom)
-		)
-	)
-	(text "Patch Bay"
-		(exclude_from_sim no)
-		(at 15.24 147.32 0)
-		(effects
-			(font
-				(size 1.27 1.27)
-			)
-			(justify left bottom)
-		)
-	)
-	(text "Cirque trackpad LH (Optional)\n"
-		(exclude_from_sim no)
-		(at 74.93 88.9 0)
-		(effects
-			(font
-				(size 1.27 1.27)
-			)
-			(justify left bottom)
-		)
-	)
-	(text "OPTIONAL decoupling 0805\n"
-		(exclude_from_sim no)
-		(at 88.265 50.165 0)
-		(effects
-			(font
-				(size 1.27 1.27)
-			)
-			(justify left bottom)
-		)
-	)
-	(text "3.5.5 SCH Change Notes:\nI2C Pin Heaqders power pin now 3V3 \nAdded GND pin to J5.5  \nAll spare GPIO to patch bay"
-		(exclude_from_sim no)
-		(at 15.24 180.34 0)
-		(effects
-			(font
-				(size 1.27 1.27)
-			)
-			(justify left bottom)
-			(href "#1")
-		)
-	)
 	(label "3V3_EN"
 		(at 50.165 158.115 180)
-		(fields_autoplaced yes)
 		(effects
 			(font
@@
 	(label "3V3_EN"
 		(at 64.77 33.02 0)
-		(fields_autoplaced yes)
 		(effects
 			(font
@@
 			)
 		)
-		(property "Value" "MBR120VLSF "
+		(property "Value" "MBR120VLSF"
 			(at 68.58 21.59 90)
 			(effects
@@
 		)
 	)
+	(embedded_fonts no)
 )
